Commit message: tree apply force moving. sphereical joints need

File: assets/franka_description/robots/tree_test.urdf (robot description, URDF)
Before this commit: robot pi_robot, 4 links, 3 joints
Links:
- link base_link: geometry collision box size=1 1 0.02; visual box size=1 1 0.02
- link leaf1: geometry collision box size=.1 .1 .1; visual box size=.1 .1 .1
- link link1: geometry collision cylinder length=1 radius=0.1; visual cylinder length=1 radius=0.1
- link link2: geometry collision cylinder length=0.5 radius=0.05; visual cylinder length=0.5 radius=0.05

Commit message: urdf spherical

File: assets/franka_description/robots/tree_test.urdf (robot description, URDF)
Before this commit: robot pi_robot, 4 links, 3 joints
Links:
- added link link2x, mass 0.001
- added link link2z, mass 0.001
Joints:
- removed joint link2_joint
- added joint link2_jointx: type revolute, parent link1, child link2x, origin xyz=0 0 1 rpy=0 0 0, axis 1 0 0, limit lower=-3.1416 upper=3.1416 effort=10 velocity=3
- added joint link2_jointy: type revolute, parent link2x, child link2z, origin xyz=0 0 0 rpy=0 0 0, axis 1 0 0, limit lower=-3.1416 upper=3.1416 effort=10 velocity=3
- added joint link2_jointz: type revolute, parent link2z, child link2, origin xyz=0 0 0 rpy=0 0 0, axis 1 0 0, limit lower=-3.1416 upper=3.1416 effort=10 velocity=3

Commit message: 2 spherical joints tree

File: assets/franka_description/robots/tree_test.urdf (robot description, URDF)
Before this commit: robot pi_robot, 6 links, 5 joints
Links:
- added link link1x, mass 0.001
- added link link1z, mass 0.001
Joints:
- removed joint link1_joint
- added joint link1_jointx: type revolute, parent base_link, child link1x, origin xyz=0 0 0.01 rpy=0 0 0, axis 1 0 0, limit lower=-3.1416 upper=3.1416 effort=10 velocity=3
- added joint link1_jointy: type revolute, parent link1x, child link1z, origin xyz=0 0 0 rpy=0 0 0, axis 0 1 0, limit lower=-3.1416 upper=3.1416 effort=10 velocity=3
- added joint link1_jointz: type revolute, parent link1z, child link1, origin xyz=0 0 0 rpy=0 0 0, axis 0 0 1, limit lower=-3.1416 upper=3.1416 effort=10 velocity=3
- joint link2_jointy: axis 1 0 0 -> 0 1 0
- joint link2_jointz: axis 1 0 0 -> 0 0 1

Commit message: spherical joints with save data

File: assets/franka_description/robots/tree_test.urdf (robot description, URDF)
Before this commit: robot pi_robot, 8 links, 7 joints
Links:
- removed link leaf1
- added link link3; collision box size=.1 .1 .1; visual box size=.1 .1 .1
- added link link3x, mass 0.001
- added link link3z, mass 0.001
Joints:
- removed joint link3_joint
- added joint link3_jointx: type revolute, parent link2, child link3x, origin xyz=0 0 0.5 rpy=0 0 0, axis 1 0 0, limit lower=-3.1416 upper=3.1416 effort=10 velocity=3
- added joint link3_jointy: type revolute, parent link3x, child link3z, origin xyz=0 0 0 rpy=0 0 0, axis 0 1 0, limit lower=-3.1416 upper=3.1416 effort=10 velocity=3
- added joint link3_jointz: type revolute, parent link3z, child link3, origin xyz=0 0 0 rpy=0 0 0, axis 0 0 1, limit lower=-3.1416 upper=3.1416 effort=10 velocity=3

Commit message: 3d tree

File: assets/franka_description/robots/tree_test.urdf (robot description, URDF)
Before this commit: robot pi_robot, 10 links, 9 joints
Links:
- added link link4; collision cylinder length=0.5 radius=0.03; visual cylinder length=0.5 radius=0.03
- added link link4x, mass 0.001
- added link link4z, mass 0.001
- link link3: geometry collision cylinder length=0.5 radius=0.04; visual cylinder length=0.5 radius=0.04
Joints:
- added joint link4_jointx: type revolute, parent link3, child link4x, origin xyz=0 0 0.5 rpy=0 0 0, axis 1 0 0, limit lower=-3.1416 upper=3.1416 effort=10 velocity=3
- added joint link4_jointy: type revolute, parent link4x, child link4z, origin xyz=0 0 0 rpy=0 0 0, axis 0 1 0, limit lower=-3.1416 upper=3.1416 effort=10 velocity=3
- added joint link4_jointz: type revolute, parent link4z, child link4, origin xyz=0 0 0 rpy=0 0 0, axis 0 0 1, limit lower=-3.1416 upper=3.1416 effort=10 velocity=3

Commit message: tree recent

File: assets/franka_description/robots/tree_test.urdf (robot description, URDF)
Before this commit: robot pi_robot, 13 links, 12 joints
Links:
- added link link5; collision cylinder length=0.5 radius=0.03; visual cylinder length=0.5 radius=0.03
- added link link6; collision cylinder length=0.5 radius=0.03; visual cylinder length=0.5 radius=0.03
- added link link7; collision cylinder length=0.5 radius=0.04; visual cylinder length=0.5 radius=0.02
- added link link7x, mass 0.001
- added link link7z, mass 0.001
- added link link8; collision cylinder length=0.5 radius=0.04; visual cylinder length=0.5 radius=0.02
- added link link9; collision cylinder length=0.5 radius=0.04; visual cylinder length=0.5 radius=0.02
- added link link9x, mass 0.001
- added link link9z, mass 0.001
Joints:
- added joint link5_jointz: type revolute, parent link4z, child link5, origin xyz=0 0 0 rpy=0 0 0, axis 0 0 1, limit lower=-3.1416 upper=3.1416 effort=10 velocity=3
- added joint link6_jointz: type revolute, parent link4z, child link6, origin xyz=0 0 0 rpy=0 0 0, axis 0 0 1, limit lower=-3.1416 upper=3.1416 effort=10 velocity=3
- added joint link7_jointx: type revolute, parent link4, child link7x, origin xyz=0.35355339058 -0.25 0.25 rpy=0 0 0, axis 1 0 0, limit lower=-3.1416 upper=3.1416 effort=10 velocity=3
- added joint link7_jointy: type revolute, parent link7x, child link7z, origin xyz=0 0 0 rpy=0 0 0, axis 0 1 0, limit lower=-3.1416 upper=3.1416 effort=10 velocity=3
- added joint link7_jointz: type revolute, parent link7z, child link7, origin xyz=0 0 0 rpy=0 0 0, axis 0 0 1, limit lower=-3.1416 upper=3.1416 effort=10 velocity=3
- added joint link8_jointz: type revolute, parent link7z, child link8, origin xyz=0 0 0 rpy=0 0 0, axis 0 0 1, limit lower=-3.1416 upper=3.1416 effort=10 velocity=3
- added joint link9_jointx: type revolute, parent link5, child link9x, origin xyz=0.35355339058 -0.25 0.25 rpy=0 0 0, axis 1 0 0, limit lower=-3.1416 upper=3.1416 effort=10 velocity=3
- added joint link9_jointy: type revolute, parent link9x, child link9z, origin xyz=0 0 0 rpy=0 0 0, axis 0 1 0, limit lower=-3.1416 upper=3.1416 effort=10 velocity=3
- added joint link9_jointz: type revolute, parent link9z, child link9, origin xyz=0 0 0 rpy=0 0 0, axis 0 0 1, limit lower=-3.1416 upper=3.1416 effort=10 velocity=3

Commit message: separated tree test and full

File: assets/franka_description/robots/tree_test.urdf (robot description, URDF)
Before this commit: robot pi_robot, 22 links, 21 joints
Links:
- removed link link4
- removed link link4x
- removed link link4z
- removed link link5
- removed link link6
- removed link link7
- removed link link7x
- removed link link7z
- removed link link8
- removed link link9
- removed link link9x
- removed link link9z
- link link3: geometry collision box size=.1 .1 .1; visual box size=.1 .1 .1
Joints:
- removed joint link4_jointx
- removed joint link4_jointy
- removed joint link4_jointz
- removed joint link5_jointz
- removed joint link6_jointz
- removed joint link7_jointx
- removed joint link7_jointy
- removed joint link7_jointz
- removed joint link8_jointz
- removed joint link9_jointx
- removed joint link9_jointy
- removed joint link9_jointz
