Commit message: reverting back to correct RPY without errors

File: assets/franka_description/robots/tree_full.urdf (robot description, URDF)
Before this commit: robot pi_robot, 33 links, 32 joints
Links:
- link link10: geometry collision cylinder length=0.5 radius=0.02; visual cylinder length=0.5 radius=0.02
- link link11: geometry collision cylinder length=0.5 radius=0.02; visual cylinder length=0.5 radius=0.02
- link link3: geometry collision cylinder length=0.5 radius=0.05; visual cylinder length=0.5 radius=0.05
- link link4: geometry collision cylinder length=0.05 radius=0.003; visual cylinder length=0.5 radius=0.03
- link link7: geometry collision cylinder length=0.5 radius=0.02; visual cylinder length=0.5 radius=0.02
- link link8: geometry collision cylinder length=0.5 radius=0.02; visual cylinder length=0.5 radius=0.02
Joints:
- joint link11L: origin xyz=-0.3535533906 0.25 0.25 rpy=0 0 0 -> xyz=-0.25 0.35355339058 0.25 rpy=0 0 0
- joint link11_jointx: origin xyz=-0.35355339058 0.25 0.25 rpy=0 0 0 -> xyz=-0.25 0.35355339058 0.25 rpy=0 0 0
- joint link7L: origin xyz=0.3535533906 -0.25 0.25 rpy=0 0 0 -> xyz=0.25 -0.3535533906 0.25 rpy=0 0 0
- joint link7_jointx: origin xyz=0.35355339058 -0.25 0.25 rpy=0 0 0 -> xyz=0.25 -0.3535533906 0.25 rpy=0 0 0
- joint link9L: origin xyz=-0.3535533906 -0.25 0.25 rpy=0 0 0 -> xyz=-0.25 -0.35355339058  0.25 rpy=0 0 0
- joint link9_jointx: origin xyz=-0.35355339058 -0.25 0.25 rpy=0 0 0 -> xyz=-0.25 -0.35355339058  0.25 rpy=0 0 0
